File: Hardware/BreakoutBoard/PCB/BreakoutBoard/BreakoutBoard.kicad_sch (KiCad schematic)
At the start: 14 parts, among them J1 Conn_01x20_Female, J10 Barrel_Jack, J11 Conn_01x08_Male, J12 Conn_01x08_Male, J13 Conn_01x08_Male, J2 Conn_01x20_Female, J3 1502_01, J4 1502_01, J5 Conn_01x04_Male, J6 Conn_01x04_Male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

Commit message: Updated schematic annotations and README.md
Other:
- title: (none) -> Daisy Seed Development Kit Breakout Board
Changed lines of the file:
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@@
 (kicad_sch (version 20211123) (generator eeschema)
   (paper "A4")
+  (title_block
+    (title "Daisy Seed Development Kit Breakout Board")
+    (date "2023-11-05")
+    (rev "1.0.1")
+  )
   (junction (at 95.25 137.16) (diameter 0) (color 0 0 0 0)
   )
