File: Hardware/Midi/PCB/Midi/Midi.kicad_sch (KiCad schematic)
At the start: 10 parts, among them J1 Conn_01x04_Male, J2 DIN-5_180degree, J3 DIN-5_180degree, U1 H11L1

Commit message: Updated schematic annotations and README.md
Other:
- title: (none) -> Daisy Seed Development Kit Midi Adapter
Changed lines of the file:
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@@
 (kicad_sch (version 20211123) (generator eeschema)
   (paper "A4")
+  (title_block
+    (title "Daisy Seed Development Kit Midi Adapter")
+    (date "2023-11-05")
+    (rev "1.0.1")
+  )
   (junction (at 119.38 82.55) (diameter 0) (color 0 0 0 0)
   )
