File: Hardware/PotentiometerArray/PCB/PotentiometerArray/PotentiometerArray.kicad_sch (KiCad schematic)
At the start: 19 parts, among them J1 Conn_01x08_Male, U1 CD4051B, U2 CD4051B

Commit message: Updated schematic annotations and README.md
Other:
- title: (none) -> Daisy Seed Development Kit Potentiometer Array
Changed lines of the file:
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@@
 (kicad_sch (version 20211123) (generator eeschema)
   (paper "A4")
+  (title_block
+    (title "Daisy Seed Development Kit Potentiometer Array")
+    (date "2023-11-05")
+    (rev "1.0.1")
+  )
   (junction (at 140.97 58.42) (diameter 0) (color 0 0 0 0)
   )
