File: Hardware/ExternalCodec/PCB/ExternalCodec/ExternalCodec.kicad_pcb (KiCad board)
At the start: 2 copper layers, 78.7 x 53.3 mm, 26 parts, among them J1 Conn_01x08_Male, J2 Conn_01x04_Male, J3 Conn_01x06_Male, J4 AudioJack3, J5 AudioJack3, J6 Conn_01x14_Female, J7 Conn_01x14_Female, U1 WM8731SEDS

Commit message: ExternalCodec drivers added
Other:
- board text added: "EXTERNAL CODEC"
Changed lines of the file:
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@@
+    (effects (font (size 1 1) (thickness 0.15)))
+  )
+  (gr_text "EXTERNAL CODEC" (at 146.05 110.49) (layer "F.SilkS")
     (effects (font (size 1 1) (thickness 0.15)))
   )
