File: Hardware/StepSequencer/PCB/StepSequencer/StepSequencer.kicad_pcb (KiCad board)
At the start: 2 copper layers, 188 x 68.8 mm, 72 parts, among them J1 Conn_01x04_Male, U1 MCP23017_SP, U2 MCP23017_SP

Commit message: Hardware update
Parts:
- removed Dx31: LED, LED_THT:LED_D3.0mm
- removed Dx37: 1N4148, Diode_THT:D_DO-35_SOD27_P7.62mm_Horizontal
- removed SWx19: SW_DIP_x01, Button_Switch_THT:SW_PUSH_6mm
- moved SW23 253.4 mm to (167.3, 108.5), turned to -90 degrees
- moved SW17 253.0 mm to (144.5, 108.5), turned to -90 degrees
- moved SW20 233.3 mm to (157.2, 95.2), turned to -90 degrees
- moved SW21 218.9 mm to (167.3, 95.2), turned to -90 degrees
- moved SW22 216.5 mm to (157.2, 108.5), turned to -90 degrees
- moved SW15 205.3 mm to (134.3, 108.5), turned to -90 degrees
- moved R6 203.2 mm to (83.8, 61.0), turned to -90 degrees
- moved SW10 199.7 mm to (103.8, 108.5), turned to -90 degrees
- moved SW8 191.5 mm to (93.7, 108.5), turned to -90 degrees
- moved SW6 187.0 mm to (83.5, 108.5), turned to -90 degrees
- moved R7 185.6 mm to (87.6, 61.0), turned to -90 degrees
- moved R8 176.1 mm to (91.4, 61.0), turned to -90 degrees
- moved SW13 175.6 mm to (124.2, 108.5), turned to -90 degrees
- moved SW12 175.5 mm to (114.0, 108.5), turned to -90 degrees
- moved R4 173.3 mm to (76.2, 61.0), turned to -90 degrees
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- renumbered Dx26 to D1, Dx36 to D10, Dx22 to D11, Dx35 to D12, Dx34 to D13, Dx23 to D14, Dx33 to D15, Dx24 to D16, Dx32 to D17, Dx1 to D18, Dx2 to D19, Dx25 to D2, Dx3 to D20, Dx4 to D21, Dx5 to D22, Dx6 to D23, Dx12 to D24, Dx11 to D25, Dx10 to D26, Dx9 to D27, Dx8 to D28, Dx7 to D29, Dx27 to D3, Dx13 to D30, Dx14 to D31, Dx15 to D32, Dx16 to D33, Dx17 to D34, Dx18 to D35, Dx19 to D4, Dx28 to D5, Dx29 to D6, Dx20 to D7, Dx30 to D8, Dx21 to D9, Rx6 to R3, Rx5 to R4, Rx4 to R5, Rx1 to R6, Rx2 to R7, Rx3 to R8, SWx9 to SW1, SWx15 to SW10, SWx5 to SW11, SWx16 to SW12, SWx17 to SW13, SWx4 to SW14, SWx18 to SW15, SWx3 to SW16, SWx24 to SW17, SWx2 to SW18, SWx1 to SW19, SWx10 to SW2, SWx20 to SW20, SWx21 to SW21, SWx23 to SW22, SWx22 to SW23, SWx8 to SW3, SWx11 to SW4, SWx7 to SW5, SWx13 to SW6, SWx12 to SW7, SWx14 to SW8, SWx6 to SW9
Connections:
- R3 pad 1: GPAx6 -> GPA2
- R4 pad 1: GPAx5 -> GPA3
- R5 pad 1: GPAx4 -> GPA4
- R6 pad 1: GPAx1 -> GPA5
- R7 pad 1: GPAx2 -> GPA6
- R8 pad 1: GPAx3 -> GPA7
- SW1 pad 1: GPCx2 -> GPC5
- SW1 pad 2: GPD2 -> GPD3
- SW10 pad 1: GPCx3 -> GPC6
- SW10 pad 2: GPD2 -> GPD3
- SW11 pad 1: GPCx1 -> GPC4
- SW11 pad 2: unconnected-(SWx5-Pad2) -> GPD1
- SW12 pad 1: GPCx3 -> GPC6
- SW12 pad 2: GPD3 -> GPD2
- SW13 pad 1: GPCx3 -> GPC6
- SW13 pad 2: unconnected-(SWx17-Pad2) -> GPD1
- SW14 pad 1: GPCx1 -> GPC4
- SW14 pad 2: GPD3 -> GPD2
- SW15 pad 1: GPCx3 -> GPC6
- SW15 pad 2: GPD5 -> GPD0
- SW16 pad 1: GPCx1 -> GPC4
- SW16 pad 2: unconnected-(SWx3-Pad2) -> GPD3
- SW17 pad 1: GPCx4 -> GPC7
- SW17 pad 2: GPD5 -> GPD0
- SW18 pad 1: GPCx1 -> GPC4
- SW18 pad 2: unconnected-(SWx2-Pad2) -> GPD4
- SW19 pad 1: GPCx1 -> GPC4
- SW19 pad 2: Net-(SWx1-Pad2) -> GPD5
- SW2 pad 1: GPCx2 -> GPC5
- SW2 pad 2: GPD3 -> GPD2
- SW20 pad 1: GPCx4 -> GPC7
- SW20 pad 2: GPD1 -> GPD4
- SW21 pad 1: GPCx4 -> GPC7
- SW21 pad 2: GPD2 -> GPD3
- SW22 pad 1: GPCx4 -> GPC7
- SW22 pad 2: unconnected-(SWx23-Pad2) -> GPD1
- SW23 pad 1: GPCx4 -> GPC7
- SW23 pad 2: GPD3 -> GPD2
- SW3 pad 1: GPCx2 -> GPC5
- SW3 pad 2: GPD1 -> GPD4
- SW4 pad 1: GPCx2 -> GPC5
- SW4 pad 2: unconnected-(SWx11-Pad2) -> GPD1
- SW5 pad 1: GPCx2 -> GPC5
- SW5 pad 2: GPD0 -> GPD5
- SW6 pad 1: GPCx3 -> GPC6
- SW6 pad 2: GPD0 -> GPD5
- SW7 pad 1: GPCx2 -> GPC5
- SW7 pad 2: GPD5 -> GPD0
- SW8 pad 1: GPCx3 -> GPC6
- SW8 pad 2: GPD1 -> GPD4
- SW9 pad 1: GPCx1 -> GPC4
- SW9 pad 2: unconnected-(SWx6-Pad2) -> GPD0
Routing:
- net GPD4: track 0.00 -> 339.7 mm
- net GPD3: track 0.00 -> 323.5 mm
- net GPD2: track 0.00 -> 323.2 mm
- net GPD1: track 0.00 -> 309.4 mm
- net GPC5: track 0.00 -> 291.7 mm
- net GPD0: track 39.8 -> 297.5 mm
- net GPD5: track 0.00 -> 230.4 mm
- net GPC6: track 0.00 -> 167.7 mm
- net Net-(D17-Pad2): track 0.00 -> 161.5 mm, vias 0 -> 2
- net Net-(D4-Pad2): track 0.00 -> 146.0 mm
- net GPC4: track 0.00 -> 144.2 mm
- net Net-(D2-Pad2): track 0.00 -> 120.0 mm, vias 0 -> 2
- net 3V3_D: track 0.00 -> 115.6 mm
- net GPC7: track 0.00 -> 113.1 mm
- net SCL: track 0.00 -> 93.3 mm
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- added copper zone on B.Cu, net GND
Other:
- board size 188 x 68.8 mm -> 132.1 x 63.5 mm
- board text added: "1"
- board text added: "10"
- board text added: "11"
- board text added: "12"
- board text added: "13"
- board text added: "14"
- board text added: "15"
- board text added: "16"
- board text added: "2"
- board text added: "3"
- board text added: "3V3_D"
- board text added: "4"
- board text added: "5"
- board text added: "6"
- board text added: "7"
- board text added: "8"
- board text added: "9"
- board text added: "A"
- board text added: "A#"
- board text added: "ACCENT"
- board text added: "B"
- board text added: "BACK"
- board text added: "C"
- board text added: "C#"
- board text added: "D"
- board text added: "D#"
- board text added: "E"
- board text added: "F"
- board text added: "F#"
- board text added: "FUNC"
- board text added: "G"
- board text added: "G#"
- board text added: "GND"
- board text added: "NEXT"
- board text added: "OCT+"
- board text added: "OCT-"
- board text added: "PATTERN"
- board text added: "PLAY"
- board text added: "REC"
- board text added: "SCL"
- board text added: "SDA"
- board text added: "SLIDE"
- board text removed: "play"
- board text removed: "rec"
