File: Hardware/StepSequencer/PCB/StepSequencer/StepSequencer.kicad_pcb (KiCad board)
At the start: 2 copper layers, 132.1 x 63.5 mm, 69 parts, among them J1 Conn_01x04_Male, SW1 SW_DIP_x01, SW10 SW_DIP_x01, SW11 SW_DIP_x01, SW12 SW_DIP_x01, SW13 SW_DIP_x01, SW14 SW_DIP_x01, SW15 SW_DIP_x01, SW16 SW_DIP_x01, SW17 SW_DIP_x01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

Commit message: General refactoring
Other:
- board text added: "STEP SEQUENCER"
- board text removed: "STEP SEQUENCER INTERFACE"
Changed lines of the file:
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@@
   (paper "A4")
   (title_block
-    (title "Daisy Seed Development Kit Step Sequencer Interface")
+    (title "Daisy Seed Development Kit Step Sequencer")
     (date "2024-01-22")
     (rev "2.0")
@@
     (effects (font (size 1 1) (thickness 0.15)))
   )
-  (gr_text "STEP SEQUENCER INTERFACE" (at 168.91 72.43) (layer "F.SilkS")
+  (gr_text "STEP SEQUENCER" (at 168.91 72.43) (layer "F.SilkS")
     (effects (font (size 1 1) (thickness 0.15)) (justify right))
   )

Commit message: Configured drivers to new hardware
Parts:
- R3, R4, R5, R6, R7, R8: value 20Ω -> 200Ω
