File: Hardware/StepSequencerInterface/PCB/StepSequencerInterface/StepSequencerInterface.kicad_sch (KiCad schematic)
At the start: 69 parts, among them J1 Conn_01x04_Male, SW1 SW_DIP_x01, SW10 SW_DIP_x01, SW11 SW_DIP_x01, SW12 SW_DIP_x01, SW13 SW_DIP_x01, SW14 SW_DIP_x01, SW15 SW_DIP_x01, SW16 SW_DIP_x01, SW17 SW_DIP_x01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

Commit message: Finished interface and renaming
Other:
- title: Daisy Seed Development Kit Step Sequencer -> Daisy Seed Development Kit Step Sequencer Interface
Changed lines of the file:
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@@
   (paper "A4")
   (title_block
-    (title "Daisy Seed Development Kit Step Sequencer")
-    (date "2024-01-17")
+    (title "Daisy Seed Development Kit Step Sequencer Interface")
+    (date "2024-01-22")
     (rev "2.0")
   )
