File: Hardware/StepSequencerInterface/PCB/StepSequencerInterface/StepSequencerInterface.kicad_pcb (KiCad board)
At the start: 2 copper layers, 132.1 x 63.5 mm, 69 parts, among them J1 Conn_01x04_Male, SW1 SW_DIP_x01, SW10 SW_DIP_x01, SW11 SW_DIP_x01, SW12 SW_DIP_x01, SW13 SW_DIP_x01, SW14 SW_DIP_x01, SW15 SW_DIP_x01, SW16 SW_DIP_x01, SW17 SW_DIP_x01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

Commit message: Finished interface and renaming
Other:
- board text added: "STEP SEQUENCER INTERFACE"
Changed lines of the file:
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@@
   (paper "A4")
   (title_block
-    (title "Daisy Seed Development Kit Step Sequencer")
-    (date "2023-12-03")
-    (rev "1.0")
+    (title "Daisy Seed Development Kit Step Sequencer Interface")
+    (date "2024-01-22")
+    (rev "2.0")
   )
   (layers
@@
     (fp_line (start 6.25 5.25) (end 0.25 5.25) (layer "F.Fab") (width 0.1))
     (fp_line (start 0.25 5.25) (end 0.25 -0.75) (layer "F.Fab") (width 0.1))
-    (fp_line (start 3.25 -0.75) (end 6.25 -0.75) (layer "F.Fab") (width 0.1))
     (fp_line (start 0.25 -0.75) (end 3.25 -0.75) (layer "F.Fab") (width 0.1))
+    (fp_line (start 3.25 -0.75) (end 6.25 -0.75) (layer "F.Fab") (width 0.1))
     (fp_line (start 6.25 -0.75) (end 6.25 5.25) (layer "F.Fab") (width 0.1))
     (fp_circle (center 3.25 2.25) (end 1.25 2.5) (layer "F.Fab") (width 0.1) (fill none))
@@
     (effects (font (size 1 1) (thickness 0.15)))
   )
+  (gr_text "STEP SEQUENCER INTERFACE" (at 168.91 72.43) (layer "F.SilkS")
+    (effects (font (size 1 1) (thickness 0.15)) (justify right))
+  )
   (gr_text "BACK" (at 154.94 117.134) (layer "F.SilkS")

Commit message: Refactor of BassSeed
Routing:
- net GPC5: track 291.7 -> 290.3 mm
Changed lines of the file:
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@@
   (segment (start 148.14048 102.08952) (end 148.14048 95.42202) (width 0.25) (layer "B.Cu") (net 47))
   (segment (start 63.21 108.55) (end 63.21 115.05) (width 0.25) (layer "B.Cu") (net 47))
+  (segment (start 152.082501 91.48) (end 167.004282 91.48) (width 0.25) (layer "B.Cu") (net 47))
   (segment (start 53.05 108.55) (end 53.05 115.05) (width 0.25) (layer "B.Cu") (net 47))
   (segment (start 66.46 97.83) (end 59.96 97.83) (width 0.25) (layer "B.Cu") (net 47))
-  (segment (start 148.14048 97.83) (end 148.14048 95.422021) (width 0.25) (layer "B.Cu") (net 47))
+  (segment (start 88.61 96) (end 90.88952 98.27952) (width 0.25) (layer "B.Cu") (net 47))
   (segment (start 73.37 108.55) (end 73.37 115.05) (width 0.25) (layer "B.Cu") (net 47))
   (segment (start 86.78 97.83) (end 70.12 97.83) (width 0.25) (layer "B.Cu") (net 47))
-  (segment (start 148.14048 95.422021) (end 152.082501 91.48) (width 0.25) (layer "B.Cu") (net 47))
   (segment (start 88.61 96) (end 86.78 97.83) (width 0.25) (layer "B.Cu") (net 47))
   (segment (start 54.88 116.88) (end 61.38 116.88) (width 0.25) (layer "B.Cu") (net 47))
   (segment (start 143.95952 106.27048) (end 148.14048 102.08952) (width 0.25) (layer "B.Cu") (net 47))
-  (segment (start 167.004282 91.48) (end 169.99452 88.489762) (width 0.25) (layer "B.Cu") (net 47))
-  (segment (start 90.88952 98.27952) (end 147.69096 98.27952) (width 0.25) (layer "B.Cu") (net 47))
-  (segment (start 169.98452 73.535956) (end 168.058084 71.60952) (width 0.25) (layer "B.Cu") (net 47))
   (segment (start 88.61 89.5) (end 88.61 96) (width 0.25) (layer "B.Cu") (net 47))
   (segment (start 75.64952 106.27048) (end 143.95952 106.27048) (width 0.25) (layer "B.Cu") (net 47))
-  (segment (start 152.082501 91.48) (end 167.004282 91.48) (width 0.25) (layer "B.Cu") (net 47))
   (segment (start 53.05 115.05) (end 54.88 116.88) (width 0.25) (layer "B.Cu") (net 47))
+  (segment (start 169.99452 88.489762) (end 169.99452 84.056197) (width 0.25) (layer "B.Cu") (net 47))
+  (segment (start 70.12 97.83) (end 68.29 96) (width 0.25) (layer "B.Cu") (net 47))
+  (segment (start 164.24952 71.60952) (end 162.54 69.9) (width 0.25) (layer "B.Cu") (net 47))
   (segment (start 168.058084 71.60952) (end 164.24952 71.60952) (width 0.25) (layer "B.Cu") (net 47))
-  (segment (start 70.12 97.83) (end 68.29 96) (width 0.25) (layer "B.Cu") (net 47))
-  (segment (start 169.99452 84.056197) (end 169.98452 84.046197) (width 0.25) (layer "B.Cu") (net 47))
-  (segment (start 88.61 96) (end 90.88952 98.27952) (width 0.25) (layer "B.Cu") (net 47))
-  (segment (start 169.98452 84.046197) (end 169.98452 73.535956) (width 0.25) (layer "B.Cu") (net 47))
-  (segment (start 169.99452 88.489762) (end 169.99452 84.056197) (width 0.25) (layer "B.Cu") (net 47))
   (segment (start 71.54 116.88) (end 73.37 115.05) (width 0.25) (layer "B.Cu") (net 47))
   (segment (start 68.29 89.5) (end 68.29 96) (width 0.25) (layer "B.Cu") (net 47))
-  (segment (start 164.24952 71.60952) (end 162.54 69.9) (width 0.25) (layer "B.Cu") (net 47))
+  (segment (start 167.004282 91.48) (end 169.99452 88.489762) (width 0.25) (layer "B.Cu") (net 47))
   (segment (start 65.04 116.88) (end 71.54 116.88) (width 0.25) (layer "B.Cu") (net 47))
-  (segment (start 147.69096 98.27952) (end 148.14048 97.83) (width 0.25) (layer "B.Cu") (net 47))
+  (segment (start 169.98452 73.535956) (end 168.058084 71.60952) (width 0.25) (layer "B.Cu") (net 47))
+  (segment (start 145.28298 98.27952) (end 152.082501 91.48) (width 0.25) (layer "B.Cu") (net 47))
+  (segment (start 169.98452 84.046197) (end 169.98452 73.535956) (width 0.25) (layer "B.Cu") (net 47))
   (segment (start 61.38 116.88) (end 63.21 115.05) (width 0.25) (layer "B.Cu") (net 47))
+  (segment (start 169.99452 84.056197) (end 169.98452 84.046197) (width 0.25) (layer "B.Cu") (net 47))
   (segment (start 58.13 89.5) (end 58.13 96) (width 0.25) (layer "B.Cu") (net 47))
   (segment (start 68.29 96) (end 66.46 97.83) (width 0.25) (layer "B.Cu") (net 47))
+  (segment (start 90.88952 98.27952) (end 145.28298 98.27952) (width 0.25) (layer "B.Cu") (net 47))
   (segment (start 63.21 115.05) (end 65.04 116.88) (width 0.25) (layer "B.Cu") (net 47))
   (segment (start 73.37 108.55) (end 75.64952 106.27048) (width 0.25) (layer "B.Cu") (net 47))
