File: Hardware/ExternalCodec/Pcm3060/PCB/ExternalCodecPcm3060/ExternalCodecPcm3060.kicad_sch (KiCad schematic)
At the start: 29 parts, among them J1 Conn_01x02_Pin, J2 Conn_01x02_Pin, U1 PCM3060

Commit message: Updated to PCM3060
Parts:
- removed J2: Conn_01x02_Pin, symbol Connector:Conn_01x02_Pin
- removed J?: Conn_01x06_Male, Connector_PinSocket_2.54mm:PinSocket_1x06_P2.54mm_Vertical, symbol Connector:Conn_01x06_Male
- added J7: Conn_01x06_Pin, Connector_PinSocket_2.54mm:PinSocket_1x06_P2.54mm_Vertical, symbol Connector:Conn_01x06_Pin
- added J8: Conn_01x02_Pin, Connector_PinSocket_2.54mm:PinSocket_1x02_P2.54mm_Vertical, symbol Connector:Conn_01x02_Pin
- J2: renamed from J1; footprint (none) -> Connector_PinSocket_2.54mm:PinSocket_1x02_P2.54mm_Vertical
- J5, J6: renamed from J?; footprint Protoplasma.pretty:PJ-307 -> Protoplasma:PJ-307
- gave numbers to parts that had none: 10
- renumbered C3 to C1, C4 to C2, C7 to C3, C5 to C4, C8 to C5, R3 to R1, R5 to R10, R1 to R2, R2 to R4, R6 to R7, R7 to R8, R4 to R9
Connections:
- net 5V: now also J8.2 (Pin_2)
- net AUDIO_IN_L: now also J7.2 (Pin_2)
- net AUDIO_IN_R: now also J7.3 (Pin_3)
- net AUDIO_OUT_L: now also J7.4 (Pin_4)
- net AUDIO_OUT_R: now also J7.5 (Pin_5)
- net CODEC_VCOM: now also J7.6 (Pin_6)
- net GND: now also J7.1 (Pin_1), J8.1 (Pin_1)
Other:
- moved on the sheet: C10, C7, C8, C9, R10, R5, R6, R7, R8, R9
