File: Hardware/PowerSupplies/Ld1117/PCB/PowerSupplyLd1117/PowerSupplyLd1117.kicad_pcb (KiCad board)
At the start: 2 copper layers, 6 parts, among them J1 Barrel_Jack, J2 Conn_01x02_Pin, U1 LD1117S50TR_SOT223

Commit message: Added consistency
Parts:
- moved C1 30.9 mm to (84.5, 83.8)
- moved J2 30.8 mm to (99.1, 81.3), turned to 180 degrees
- moved D1 24.6 mm to (81.3, 83.8), turned to 90 degrees
- moved J1 19.6 mm to (77.5, 80.0), turned to -90 degrees
- moved U1 12.5 mm to (87.6, 78.1)
- moved C2 11.6 mm to (90.2, 83.8)
Routing:
- net /5V: track 0.00 -> 22.7 mm
- net /7-15V: track 0.00 -> 11.7 mm
- net Net-(D1-K): track 0.00 -> 6.64 mm
- added copper zone on F.Cu, net GND
Other:
- board outline added: 38.1 x 12.7 mm
- board text added: "5V"
- board text added: "GND"
- board text added: "LD1117 PSU"
