File: Hardware/PowerSupplies/Lm7805/PCB/PowerSupplyLm7805/PowerSupplyLm7805.kicad_pcb (KiCad board)
At the start: 2 copper layers, 7 parts, among them J1 Conn_01x02_Pin, J2 Barrel_Jack, U1 LM7805_TO220

Commit message: Added consistency
Parts:
- added D1: BAT43, Diode_THT:D_DO-35_SOD27_P7.62mm_Horizontal, F.Cu at (88.3, 85.1)
- C1: value 330μF -> 10μF; footprint Capacitor_THT:C_Disc_D5.0mm_W2.5mm_P2.50mm -> Capacitor_THT:C_Radial_D6.3mm_H7.0mm_P2.50mm
- C2: value 100μF -> 330nF; footprint Capacitor_THT:C_Disc_D5.0mm_W2.5mm_P2.50mm -> Capacitor_THT:C_Disc_D5.0mm_W2.5mm_P5.00mm
- C3: value 10μF -> 100nF; footprint Capacitor_THT:C_Radial_D6.3mm_H7.0mm_P2.50mm -> Capacitor_THT:C_Disc_D5.0mm_W2.5mm_P2.50mm
- moved C1 35.9 mm to (94.0, 82.0), turned to -90 degrees
- moved J2 29.9 mm to (85.0, 81.3), turned to -90 degrees
- moved C2 29.0 mm to (96.5, 77.5), turned to 180 degrees
- moved C3 25.7 mm to (106.0, 85.1)
- moved C4 13.9 mm to (106.0, 79.8)
- moved J1 11.5 mm to (114.3, 82.6), turned to 180 degrees
- moved U1 3.08 mm to (99.7, 78.7), turned to -90 degrees
Connections:
- C1 pad 1: /7-35V -> Net-(D1-K)
- C2 pad 1: /5V -> Net-(D1-K)
- C3 pad 1: /7-35V -> /5V
- U1 pad 1: /7-35V -> Net-(D1-K)
Routing:
- net /5V: track 0.00 -> 23.6 mm
- net Net-(D1-K): track 0.00 -> 15.6 mm
- net /7-35V: track 0.00 -> 11.1 mm
- added copper zone on F.Cu, net GND
Other:
- board outline added: 47 x 12.7 mm
- board text added: "5V"
- board text added: "GND"
- board text added: "LM7805 PSU"
