File: Hardware/PowerSupplies/Lm7805/PCB/PowerSupplyLm7805/PowerSupplyLm7805.kicad_sch (KiCad schematic)
At the start: 6 parts, among them J1 Conn_01x02_Pin, J2 Barrel_Jack, U1 LM7805_TO220

Commit message: Added consistency
Parts:
- added C2: 330nF, Capacitor_THT:C_Disc_D5.0mm_W2.5mm_P5.00mm, symbol Device:C
- added C3: 100nF, Capacitor_THT:C_Disc_D5.0mm_W2.5mm_P2.50mm, symbol Device:C
- renumbered C3 to C1
Connections:
- net 5V: now also C3.1
- net GND: now also C2.2, C3.2
- net at C1.1, D1.1 (K), U1.1 (VI): now also C2.1
Other:
- moved on the sheet: C1, C4
Changed lines of the file:
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@@
 	)
 	(junction
-		(at 160.02 82.55)
+		(at 113.03 82.55)
 		(diameter 0)
 		(color 0 0 0 0)
 	)
 	(junction
-		(at 119.38 90.17)
+		(at 125.73 82.55)
 		(diameter 0)
 		(color 0 0 0 0)
 	)
 	(junction
-		(at 119.38 82.55)
+		(at 166.37 82.55)
+		(diameter 0)
+		(color 0 0 0 0)
+	)
+	(junction
+		(at 153.67 82.55)
+		(diameter 0)
+		(color 0 0 0 0)
+	)
+	(junction
+		(at 153.67 90.17)
+		(diameter 0)
+		(color 0 0 0 0)
+	)
+	(junction
+		(at 166.37 90.17)
 		(diameter 0)
 		(color 0 0 0 0)
@@
 	)
 	(junction
-		(at 160.02 90.17)
+		(at 125.73 90.17)
 		(diameter 0)
 		(color 0 0 0 0)
 	)
-	(wire
-		(pts
-			(xy 160.02 82.55) (xy 186.69 82.55)
-		)
-		(stroke
-			(width 0)
-			(type default)
-		)
+	(junction
+		(at 113.03 90.17)
+		(diameter 0)
+		(color 0 0 0 0)
 	)
 	(wire
@@
 	(wire
 		(pts
-			(xy 147.32 82.55) (xy 160.02 82.55)
+			(xy 147.32 82.55) (xy 153.67 82.55)
 		)
 		(stroke
@@
 	(wire
 		(pts
-			(xy 90.17 90.17) (xy 119.38 90.17)
-		)
-		(stroke
-			(width 0)
-			(type default)
-		)
-	)
-	(wire
-		(pts
-			(xy 107.95 82.55) (xy 119.38 82.55)
+			(xy 90.17 90.17) (xy 113.03 90.17)
+		)
+		(stroke
+			(width 0)
+			(type default)
+		)
+	)
+	(wire
+		(pts
+			(xy 107.95 82.55) (xy 113.03 82.55)
 		)
 		(stroke
@@
 	(wire
 		(pts
-			(xy 139.7 90.17) (xy 160.02 90.17)
+			(xy 139.7 90.17) (xy 153.67 90.17)
 		)
 		(stroke
@@
 	(wire
 		(pts
-			(xy 119.38 82.55) (xy 132.08 82.55)
+			(xy 113.03 82.55) (xy 125.73 82.55)
 		)
 		(stroke
@@
 	(wire
 		(pts
-			(xy 160.02 90.17) (xy 186.69 90.17)
+			(xy 153.67 82.55) (xy 166.37 82.55)
+		)
+		(stroke
+			(width 0)
+			(type default)
+		)
+	)
+	(wire
+		(pts
+			(xy 125.73 90.17) (xy 139.7 90.17)
+		)
+		(stroke
+			(width 0)
+			(type default)
+		)
+	)
+	(wire
+		(pts
+			(xy 166.37 82.55) (xy 186.69 82.55)
 		)
 		(stroke
@@
 	(wire
 		(pts
+			(xy 113.03 90.17) (xy 125.73 90.17)
+		)
+		(stroke
+			(width 0)
+			(type default)
+		)
+	)
+	(wire
+		(pts
+			(xy 125.73 82.55) (xy 132.08 82.55)
+		)
+		(stroke
+			(width 0)
+			(type default)
+		)
+	)
+	(wire
+		(pts
+			(xy 166.37 90.17) (xy 186.69 90.17)
+		)
+		(stroke
+			(width 0)
+			(type default)
+		)
+	)
+	(wire
+		(pts
+			(xy 153.67 90.17) (xy 166.37 90.17)
+		)
+		(stroke
+			(width 0)
+			(type default)
+		)
+	)
+	(wire
+		(pts
 			(xy 88.9 88.9) (xy 90.17 88.9)
-		)
-		(stroke
-			(width 0)
-			(type default)
-		)
-	)
-	(wire
-		(pts
-			(xy 119.38 90.17) (xy 139.7 90.17)
 		)
 		(stroke
@@
 	)
 	(symbol
+		(lib_id "Device:C")
+		(at 153.67 86.36 0)
+		(unit 1)
+		(exclude_from_sim no)
+		(in_bom yes)
+		(on_board yes)
+		(dnp no)
+		(property "Reference" "C3"
+			(at 153.67 77.724 0)
+			(effects
+				(font
+					(size 1.27 1.27)
+				)
+			)
+		)
+		(property "Value" "100nF"
+			(at 153.67 80.518 0)
+			(effects
+				(font
+					(size 1.27 1.27)
+				)
+			)
+		)
+		(property "Footprint" "Capacitor_THT:C_Disc_D5.0mm_W2.5mm_P2.50mm"
+			(at 154.6352 90.17 0)
+			(effects
+				(font
+					(size 1.27 1.27)
+				)
+				(hide yes)
+			)
+		)
+		(property "Datasheet" "~"
+			(at 153.67 86.36 0)
+			(effects
+				(font
+					(size 1.27 1.27)
+				)
+				(hide yes)
+			)
+		)
+		(property "Description" ""
+			(at 153.67 86.36 0)
+			(effects
+				(font
+					(size 1.27 1.27)
+				)
+				(hide yes)
+			)
+		)
+		(pin "1"
+		)
+		(pin "2"
+		)
+		(instances
+			(project "PowerSupplyLm7805"
+				(path "/2d797758-27d9-42d0-9452-1ad0217c26de"
+					(reference "C3")
+					(unit 1)
+				)
+			)
+		)
+	)
+	(symbol
 		(lib_id "Device:C_Polarized")
-		(at 160.02 86.36 0)
+		(at 166.37 86.36 0)
 		(unit 1)
 		(exclude_from_sim no)
@@
 		(dnp no)
 		(property "Reference" "C4"
-			(at 158.496 76.454 0)
+			(at 165.1 77.724 0)
 			(effects
 				(font
@@
 		)
 		(property "Value" "10μF"
-			(at 157.48 79.756 0)
+			(at 164.084 80.264 0)
 			(effects
 				(font
@@
 		)
 		(property "Footprint" "Capacitor_THT:C_Radial_D6.3mm_H7.0mm_P2.50mm"
-			(at 160.9852 90.17 0)
+			(at 167.3352 90.17 0)
 			(effects
 				(font
@@
 		)
 		(property "Datasheet" "~"
-			(at 160.02 86.36 0)
+			(at 166.37 86.36 0)
 			(effects
 				(font
@@
 		)
 		(property "Description" "Polarized capacitor"
-			(at 160.02 86.36 0)
+			(at 166.37 86.36 0)
 			(effects
 				(font
@@
 	(symbol
 		(lib_id "Device:C_Polarized")
-		(at 119.38 86.36 0)
+		(at 113.03 86.36 0)
 		(unit 1)
 		(exclude_from_sim no)
@@
 		(on_board yes)
 		(dnp no)
-		(property "Reference" "C3"
-			(at 118.11 77.724 0)
+		(property "Reference" "C1"
+			(at 111.76 77.724 0)
 			(effects
 				(font
@@
 		)
 		(property "Value" "10μF"
-			(at 116.84 80.518 0)
+			(at 110.49 80.518 0)
 			(effects
 				(font
@@
 		)
 		(property "Footprint" "Capacitor_THT:C_Radial_D6.3mm_H7.0mm_P2.50mm"
-			(at 120.3452 90.17 0)
+			(at 113.9952 90.17 0)
 			(effects
 				(font
@@
 		)
 		(property "Datasheet" "~"
-			(at 119.38 86.36 0)
+			(at 113.03 86.36 0)
 			(effects
 				(font
@@
 		)
 		(property "Description" "Polarized capacitor"
-			(at 119.38 86.36 0)
+			(at 113.03 86.36 0)
 			(effects
 				(font
@@
 			(project "PowerSupplyLm7805"
 				(path "/2d797758-27d9-42d0-9452-1ad0217c26de"
-					(reference "C3")
+					(reference "C1")
 					(unit 1)
 				)
+			)
+		)
+	)
+	(symbol
+		(lib_id "Device:C")
+		(at 125.73 86.36 0)
+		(unit 1)
+		(exclude_from_sim no)
+		(in_bom yes)
+		(on_board yes)
+		(dnp no)
+		(property "Reference" "C2"
+			(at 125.984 77.724 0)
+			(effects
+				(font
+					(size 1.27 1.27)
+				)
+			)
+		)
+		(property "Value" "330nF"
+			(at 125.984 80.518 0)
+			(effects
+				(font
+					(size 1.27 1.27)
+				)
+			)
+		)
+		(property "Footprint" "Capacitor_THT:C_Disc_D5.0mm_W2.5mm_P5.00mm"
+			(at 126.6952 90.17 0)
+			(effects
+				(font
+					(size 1.27 1.27)
+				)
+				(hide yes)
+			)
+		)
+		(property "Datasheet" "~"
+			(at 125.73 86.36 0)
+			(effects
+				(font
+					(size 1.27 1.27)
+				)
+				(hide yes)
+			)
+		)
+		(property "Description" ""
+			(at 125.73 86.36 0)
+			(effects
+				(font
+					(size 1.27 1.27)
+				)
+				(hide yes)
+			)
+		)
+		(pin "1"
+		)
+		(pin "2"
+		)
+		(instances
+			(project "PowerSupplyLm7805"
+				(path "/2d797758-27d9-42d0-9452-1ad0217c26de"
+					(reference "C2")
+					(unit 1)
+				)
