File: Hardware/NavigationKeypad/PCB/NavigationKeypad/NavigationKeypad.kicad_pcb (KiCad board)
At the start: 2 copper layers, 43.2 x 76.2 mm, 13 parts, among them J1 Conn_01x04_Male, J2 Conn_01x04_Male, SW1 SW_DIP_x01, SW2 SW_DIP_x01, SW3 SW_DIP_x01, SW4 SW_DIP_x01, SW5 SW_DIP_x01, SW6 SW_DIP_x01, SW7 SW_DIP_x01, SW8 SW_DIP_x01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

Commit message: Removing edge and mount holes
Routing:
- net GND: track 25.0 -> 0.00 mm
- net 3V3_D: track 56.2 -> 58.9 mm
- added copper zone on B.Cu, net GND
Other:
- board size 43.2 x 76.2 mm -> 38.1 x 71.1 mm

Commit message: Finalised PCBs
Parts:
- J1: footprint Connector_PinSocket_2.54mm:PinSocket_1x04_P2.54mm_Vertical -> Connector_PinHeader_2.54mm:PinHeader_1x04_P2.54mm_Horizontal
- J2: footprint Connector_PinSocket_2.54mm:PinSocket_1x04_P2.54mm_Vertical -> Connector_PinSocket_2.54mm:PinSocket_1x04_P2.54mm_Horizontal
- moved R2 14.9 mm to (111.8, 52.7), turned to -90 degrees
- moved J2 12.1 mm to (126.4, 53.3), turned to -90 degrees
- moved J1 12.1 mm to (94.6, 53.3), turned to 90 degrees
- moved R1 9.52 mm to (108.0, 52.7), turned to -90 degrees
Connections:
- J1 pad 1: SDA -> GND
- J1 pad 2: SCL -> 3V3_D
- J1 pad 3: 3V3_D -> SCL
- J1 pad 4: GND -> SDA
- J2 pad 1: SDA -> GND
- J2 pad 2: SCL -> 3V3_D
- J2 pad 3: 3V3_D -> SCL
- J2 pad 4: GND -> SDA
Routing:
- net SDA: track 56.4 -> 45.7 mm
- net SCL: track 33.5 -> 38.2 mm
Other:
- board size 38.1 x 71.1 mm -> 38.1 x 67.6 mm
