File: Hardware/NavigationKeypad/PCB/NavigationKeypad/NavigationKeypad.kicad_sch (KiCad schematic)
At the start: 13 parts, among them J1 Conn_01x04_Male, J2 Conn_01x04_Male, SW1 SW_DIP_x01, SW2 SW_DIP_x01, SW3 SW_DIP_x01, SW4 SW_DIP_x01, SW5 SW_DIP_x01, SW6 SW_DIP_x01, SW7 SW_DIP_x01, SW8 SW_DIP_x01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

Commit message: Finalised PCBs
Parts:
- J1: footprint Connector_PinSocket_2.54mm:PinSocket_1x04_P2.54mm_Vertical -> Connector_PinHeader_2.54mm:PinHeader_1x04_P2.54mm_Horizontal
- J2: footprint Connector_PinSocket_2.54mm:PinSocket_1x04_P2.54mm_Vertical -> Connector_PinSocket_2.54mm:PinSocket_1x04_P2.54mm_Horizontal
Connections:
- net 3V3_D: now also J1.2 (Pin_2), J2.2 (Pin_2); no longer J1.3 (Pin_3), J2.3 (Pin_3)
- net GND: now also J1.1 (Pin_1), J2.1 (Pin_1); no longer J1.4 (Pin_4), J2.4 (Pin_4)
- net SCL: now also J1.3 (Pin_3), J2.3 (Pin_3); no longer J1.2 (Pin_2), J2.2 (Pin_2)
- net SDA: now also J1.4 (Pin_4), J2.4 (Pin_4); no longer J1.1 (Pin_1), J2.1 (Pin_1)
Other:
- moved on the sheet: J2
