File: Hardware/Encoder/PCB/Encoder/Encoder.kicad_sch (KiCad schematic)
At the start: 2 parts, among them J1 Conn_01x06_Male, SW1 RotaryEncoder_Switch

Commit message: Finalised PCBs
Parts:
- J1: footprint Connector_PinSocket_2.54mm:PinSocket_1x06_P2.54mm_Vertical -> Connector_PinHeader_2.54mm:PinHeader_1x06_P2.54mm_Horizontal

Commit message: Added midi and fixed unit tests
Parts:
- SW1: footprint RotaryEncoder:Bourns-PEC11R-4220F-S0024-0-0-0 -> Rotary_Encoder:RotaryEncoder_Alps_EC11E-Switch_Vertical_H20mm
Changed lines of the file:
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@@
 			)
 		)
-		(property "Footprint" "RotaryEncoder:Bourns-PEC11R-4220F-S0024-0-0-0"
+		(property "Footprint" "Rotary_Encoder:RotaryEncoder_Alps_EC11E-Switch_Vertical_H20mm"
 			(at 66.294 100.33 0)
 			(effects
